File: controller-board.kicad_sch (KiCad schematic)
At the start: 38 parts, among them J1 Conn_01x05, J2 Conn_01x05, J3 USB_C_Receptacle_USB2.0_14P, SW1 Switch, U1 ATmega32U4-A, U3 SX1280IMLTRT, Y1 16MHz, Y2 52MHz

Commit message: tweaked OLED connector
Parts:
- removed DS1: OLED-128O064D, Display:OLED-128O064D, symbol Display_Graphic:OLED-128O064D
- added C20: 10uF, symbol Device:C
- added J4: OLED Screen, symbol Connector_Generic:Conn_01x04
Connections:
- net 5V: now also C20.2, J4.2 (VDD)
- net GND: now also C20.1, J4.1 (GND)
- net SCK_OLED: now reaches U1.18 (PD0)
- net SCK_OLED: now also J4.3 (SCK)
- net SDA_OLED: now reaches U1.19 (PD1)
- net SDA_OLED: now also J4.4 (SDA)
